File: SD_Card.kicad_sch (KiCad schematic)
At the start: 14 parts, among them J1 MSD-1-A, U6 USBLC6-2SC6, U7 USBLC6-2SC6, U8 USBLC6-2SC6, U9 USBLC6-2SC6

Commit message: arranged positions of all the components
Parts:
- added C60: 22uF, Capacitor_SMD:C_0603_1608Metric_Pad1.08x0.95mm_HandSolder, symbol Device:C
- C55: footprint Capacitor_SMD:C_0805_2012Metric_Pad1.18x1.45mm_HandSolder -> Capacitor_SMD:C_0603_1608Metric_Pad1.08x0.95mm_HandSolder
Connections:
- net +3V3: now also C60.1
- net GND: now also C60.2
- net SDCO_CMD: now also U9.3 (I/O2), U9.4 (I/O2); no longer U6.1 (I/O1), U6.6 (I/O1)
- net SDCO_D0: now also U7.1 (I/O1), U7.6 (I/O1); no longer U6.3 (I/O2), U6.4 (I/O2)
- net SDCO_D1: now also U7.3 (I/O2), U7.4 (I/O2); no longer U7.1 (I/O1), U7.6 (I/O1)
- net SDCO_D2: now also U6.1 (I/O1), U6.6 (I/O1); no longer U7.3 (I/O2), U7.4 (I/O2)
- net SDCO_D3: now also U6.3 (I/O2), U6.4 (I/O2); no longer U8.3 (I/O2), U8.4 (I/O2)
