File: power.kicad_sch (KiCad schematic)
At the start: 71 parts, among them U1 MIC5501-3.0YM5, U2 TLV62569DBV, U3 TLV62569DBV, U4 TLV62569DBV

Commit message: arranged positions of all the components
Parts:
- added C58, C59: 100nF, Capacitor_SMD:C_0603_1608Metric_Pad1.08x0.95mm_HandSolder, symbol Device:C
- C1, C10, C11, C12, C13, C14, C15, C16, C17, C18, C19, C2, C20, C21, C22, C23, C24, C25, C26, C27, C28, C29, C3, C30, C31, C32, C33, C34, C35, C36, C37, C38, C39, C4, C40, C41, C42, C43, C5, C6, C7, C8, C9: footprint Capacitor_SMD:C_0805_2012Metric -> Capacitor_SMD:C_0603_1608Metric_Pad1.08x0.95mm_HandSolder
- L1, L2, L3: footprint Inductor_SMD:L_0805_2012Metric_Pad1.05x1.20mm_HandSolder -> Resistor_SMD:R_0805_2012Metric_Pad1.20x1.40mm_HandSolder
- R1, R2, R29, R3, R4, R5, R6, R7, R8: footprint Resistor_SMD:R_0805_2012Metric -> Resistor_SMD:R_0805_2012Metric_Pad1.20x1.40mm_HandSolder
Connections:
- net +3V3: now also C58.1, C59.1
- net at C34.2, C35.2, C36.2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: now also C58.2, C59.2
